Commit message: omni_6.rviz files update

File: neocobot/neo_description/urdf/omni_6/omni_6_robot.urdf.xacro (robot description, xacro)
@@ -12,5 +12,5 @@
     <parent link="world" />
     <child link = "base_link" />
-    <origin xyz="0.0 0.0 0.0" rpy="0.0 0.0 0.0" />
+    <origin xyz="0.0 0.0 0.0" rpy="0.0 0.0 -1.57" />
   </joint>
 </robot>
