Commit message: OMNI 6 - urdf update

File: neocobot/neo_description/urdf/omni_6/omni_6.urdf.xacro (robot description, xacro)
@@ -13,5 +13,5 @@
      sixth_lower_limit:=${-8.0*pi/9.0}      sixth_upper_limit:=${8.0*pi/9.0}">
 <!-- //////////////////////////////////////////////////////////////////////////////////////////////////////////// -->
-    <link name="base_link" >
+    <link name="base1_link" >
       <visual>
         <origin xyz="0 0 0" rpy="0 0 0" />
@@ -39,5 +39,5 @@
 <!-- //////////////////////////////////////////////////////////////////////////////////////////////////////////// -->
     <joint name="first_joint" type="revolute">
-      <parent link="base_link" />
+      <parent link="base1_link" />
       <child link = "first_link" />
       <origin xyz="0 0 0.1565" rpy="-5.8488E-31 0 0" />

File: neocobot/neo_description/urdf/omni_6/omni_6_robot.urdf.xacro (robot description, xacro)
@@ -8,8 +8,8 @@
   <!-- arm -->
   <xacro:omni_6_robot joint_limited="True"/>
-  <link name="world" />
+  <link name="base_footprint" />
   <joint name="world_joint" type="fixed">
-    <parent link="world" />
-    <child link = "base_link" />
+    <parent link="base_footprint" />
+    <child link = "base1_link" />
     <origin xyz="0.0 0.0 0.0" rpy="0.0 0.0 -1.57" />
   </joint>
